File: Batt_alim.sch (KiCad schematic (older format))
At the start: 5 parts, among them J4 Conn_01x02, J9 USB_B_Micro, U4 Batt_Alim

Commit message: Changement pour Batt_alim_4P version _HP
Parts:
- U4: footprint Chimere_mods:Batt_Alim -> Chimere_mods:Batt_Alim_4P_HP; symbol Chimere_mods:Batt_Alim -> Chimere_mods:Batt_Alim_4P
Changed lines of the file:
@@
 $EndDescr
 $Comp
-L Chimere_mods:Batt_Alim U4
+L Chimere_mods:Batt_Alim_4P U4
 U 1 1 5FDF7692
 P 6300 3750
@@
 F 0 "U4" H 6300 4290 50  0000 C CNN
 F 1 "Batt_Alim" H 6300 4199 50  0000 C CNN
-F 2 "Chimere_mods:Batt_Alim" H 6300 3750 50  0001 C CNN
+F 2 "Chimere_mods:Batt_Alim_4P_HP" H 6300 3750 50  0001 C CNN
 F 3 "" H 6300 3750 50  0001 C CNN
 	1    6300 3750
