File: Meca_contour.sch (KiCad schematic (older format))
At the start: 4 parts

Commit message: end of day save
Changed lines of the file:
@@
-	1    0    0    -1
-$EndComp
-$Comp
-L power:GND #PWR01
-U 1 1 5FCC214B
-P 1000 1200
-F 0 "#PWR01" H 1000 950 50  0001 C CNN
-F 1 "GND" V 1005 1072 50  0000 R CNN
-F 2 "" H 1000 1200 50  0001 C CNN
-F 3 "" H 1000 1200 50  0001 C CNN
-	1    1000 1200
 	1    0    0    -1
 $EndComp
@@
 	1    0    0    -1
 $EndComp
-$Comp
-L power:GND #PWR03
-U 1 1 5FCCD46A
-P 1000 1800
-F 0 "#PWR03" H 1000 1550 50  0001 C CNN
-F 1 "GND" V 1005 1672 50  0000 R CNN
-F 2 "" H 1000 1800 50  0001 C CNN
-F 3 "" H 1000 1800 50  0001 C CNN
-	1    1000 1800
-	1    0    0    -1
-$EndComp
 Wire Wire Line
 	1000 1750 1000 1800
@@
 F 3 "~" H 1325 1050 50  0001 C CNN
 	1    1325 1050
-	1    0    0    -1
-$EndComp
-$Comp
-L power:GND #PWR02
-U 1 1 5FCD7747
-P 1325 1200
-F 0 "#PWR02" H 1325 950 50  0001 C CNN
-F 1 "GND" V 1330 1072 50  0000 R CNN
-F 2 "" H 1325 1200 50  0001 C CNN
-F 3 "" H 1325 1200 50  0001 C CNN
-	1    1325 1200
 	1    0    0    -1
 $EndComp
@@
 	1    0    0    -1
 $EndComp
-$Comp
-L power:GND #PWR04
-U 1 1 5FCE1C3D
-P 1325 1800
-F 0 "#PWR04" H 1325 1550 50  0001 C CNN
-F 1 "GND" V 1330 1672 50  0000 R CNN
-F 2 "" H 1325 1800 50  0001 C CNN
-F 3 "" H 1325 1800 50  0001 C CNN
-	1    1325 1800
-	1    0    0    -1
-$EndComp
 Wire Wire Line
 	1325 1750 1325 1800
+Text GLabel 1000 1200 0    50   Input ~ 0
+GND
+Text GLabel 1000 1800 0    50   Input ~ 0
+GND
+Text GLabel 1325 1200 0    50   Input ~ 0
+GND
+Text GLabel 1325 1800 0    50   Input ~ 0
+GND
 $EndSCHEMATC
