File: audio.sch (KiCad schematic (older format))
At the start: 10 parts, among them J29 Conn_01x02, U1 Audio_Facile, U3 rot_pot_rot_sw

Commit message: maj split librairie
Parts:
- U1: footprint Chimere:Audio_Facile -> Chimere_mods:Audio_Facile; symbol Chimere:Audio_Facile -> Chimere_mods:Audio_Facile
- U3: footprint Chimere:PTR901 -> Chimere_comps:PTR901; symbol Chimere:rot_pot_rot_sw -> Chimere_comps:rot_pot_rot_sw
Changed lines of the file:
@@
 DAC_Rout
 $Comp
-L Chimere:Audio_Facile U1
+L Chimere_mods:Audio_Facile U1
 U 1 1 606C57A8
 P 4975 3200
@@
 F 0 "U1" H 4975 3103 50  0000 C CNN
 F 1 "Audio_Facile" H 4975 3012 50  0000 C CNN
-F 2 "Chimere:Audio_Facile" H 4975 3200 50  0001 C CNN
+F 2 "Chimere_mods:Audio_Facile" H 4975 3200 50  0001 C CNN
 F 3 "" H 4975 3200 50  0001 C CNN
 	1    4975 3200
@@
 	4025 2950 4100 2950
 $Comp
-L Chimere:rot_pot_rot_sw U3
+L Chimere_comps:rot_pot_rot_sw U3
 U 1 1 606D2DEF
 P 3225 4275
@@
 F 0 "U3" V 3515 4363 50  0000 C CNN
 F 1 "rot_pot_rot_sw" V 3424 4363 50  0000 C CNN
-F 2 "Chimere:PTR901" H 3275 4275 50  0001 C CNN
+F 2 "Chimere_comps:PTR901" H 3275 4275 50  0001 C CNN
 F 3 "" H 3275 4275 50  0001 C CNN
 	1    3225 4275

Commit message: passage à la version "HP" de audio facile
Parts:
- U1: footprint Chimere_mods:Audio_Facile -> Chimere_mods:Audio_Facile_HP
Changed lines of the file:
@@
 F 0 "U1" H 4975 3103 50  0000 C CNN
 F 1 "Audio_Facile" H 4975 3012 50  0000 C CNN
-F 2 "Chimere_mods:Audio_Facile" H 4975 3200 50  0001 C CNN
+F 2 "Chimere_mods:Audio_Facile_HP" H 4975 3200 50  0001 C CNN
 F 3 "" H 4975 3200 50  0001 C CNN
 	1    4975 3200
